File: _saved_weather_station.sch (KiCad schematic (older format))
At the start: 32 parts, among them J1 Conn_02x10_Odd_Even, J2 Conn_02x10_Odd_Even, U3 nRF52832, Y1 FL3200037

Commit message: updates
Parts:
- added C29, C30: C_Small, Capacitors_SMD:C_0402, symbol C_Small
- added J4: Conn_Coaxial, Connectors:SMA_SMD_Jack_Straight, symbol Conn_Coaxial
- added Y2: 32.786khz, Crystals:Crystal_SMD_EuroQuartz_EQ161-2pin_3.2x1.5mm, symbol Crystal
- AE1: footprint 24ghztraceantenna:PCB_IF_ANT_2.4G -> Microwave:SMA
Connections:
- net GND: now also C29.2, C30.1, J4.2 (Ext)
- net RADIO_DATA: now also U3.18 (P0.15/TRACEDATA[2]); no longer U3.17 (P0.14/TRACEDATA[3])
- net RADIO_PD: now also U3.16 (P0.13)
- net RADIO_PTT: now also U3.17 (P0.14/TRACEDATA[3]); no longer U3.16 (P0.13)
- net RADIO_UART_RX: now also U3.20 (P0.17); no longer U3.19 (P0.16/TRACEDATA[1])
- net RADIO_UART_TX: now also U3.19 (P0.16/TRACEDATA[1]); no longer U3.18 (P0.15/TRACEDATA[2])
- net ANEOMETER: now reaches U3.10 (P0.08)
- net XL1: now reaches U3.2 (P0.00/XL1)
- net XL1: now also C30.2, Y2.2
- net XL2: now reaches U3.3 (P0.01/XL2)
- net XL2: now also C29.1, Y2.1
- net at C12.2, L3.1, L4.2: now also J4.1 (In)
Changed lines of the file:
@@
 F 0 "AE1" H 7305 1345 50  0000 R CNN
 F 1 "ant" H 7305 1270 50  0001 R CNN
-F 2 "24ghztraceantenna:PCB_IF_ANT_2.4G" H 7380 1270 50  0001 C CNN
+F 2 "Microwave:SMA" H 7380 1270 50  0001 C CNN
 F 3 "" H 7380 1270 50  0001 C CNN
 	1    7380 1170
@@
 $EndComp
 Wire Wire Line
-	7740 1530 7660 1530
+	7100 1530 7740 1530
 Wire Wire Line
 	7660 1510 7660 1600
@@
 Text GLabel 10550 2900 1    60   Input ~ 0
 SWDIO
-Text GLabel 6900 4400 2    60   Input ~ 0
+Text GLabel 6900 4300 2    60   Input ~ 0
 RADIO_UART_TX
-Text GLabel 6900 4300 2    60   Input ~ 0
+Text GLabel 6900 4200 2    60   Input ~ 0
 RADIO_UART_RX
 Text GLabel 10400 4600 1    60   Input ~ 0
@@
 	0    1    1    0
 $EndComp
-Text GLabel 6900 4600 2    60   Input ~ 0
+Text GLabel 6900 4500 2    60   Input ~ 0
 RADIO_PTT
 Text GLabel 6900 2900 2    60   Input ~ 0
@@
 Entry Wire Line
 	-450 4100 -350 4200
-Text GLabel 6900 4500 2    60   Input ~ 0
+Text GLabel 6900 4400 2    60   Input ~ 0
 RADIO_DATA
 Text GLabel 6900 4700 2    60   Input ~ 0
@@
 Text GLabel 6900 3600 2    60   Input ~ 0
 SWDIO
-Text GLabel 7950 3950 2    60   Input ~ 0
+Text GLabel 6900 4600 2    60   Input ~ 0
 RADIO_PD
+$Comp
+L Crystal Y2
+U 1 1 5A788BD1
+P 2300 3550
+F 0 "Y2" H 2300 3700 50  0000 C CNN
+F 1 "32.786khz" H 2300 3400 50  0000 C CNN
+F 2 "Crystals:Crystal_SMD_EuroQuartz_EQ161-2pin_3.2x1.5mm" H 2300 3550 50  0001 C CNN
+F 3 "" H 2300 3550 50  0001 C CNN
+	1    2300 3550
+	1    0    0    -1
+$EndComp
+Text GLabel 2500 3500 1    60   Input ~ 0
+XL1
+Text GLabel 2050 3500 1    60   Input ~ 0
+XL2
+Wire Wire Line
+	2450 3550 2550 3550
+Wire Wire Line
+	2500 3550 2500 3500
+$Comp
+L C_Small C30
+U 1 1 5A7892B3
+P 2650 3550
+F 0 "C30" H 2660 3620 50  0000 L CNN
+F 1 "C_Small" H 2660 3470 50  0000 L CNN
+F 2 "Capacitors_SMD:C_0402" H 2650 3550 50  0001 C CNN
+F 3 "" H 2650 3550 50  0001 C CNN
+	1    2650 3550
+	0    1    1    0
+$EndComp
+Connection ~ 2500 3550
+$Comp
+L C_Small C29
+U 1 1 5A789395
+P 1900 3550
+F 0 "C29" H 1910 3620 50  0000 L CNN
+F 1 "C_Small" H 1910 3470 50  0000 L CNN
+F 2 "Capacitors_SMD:C_0402" H 1900 3550 50  0001 C CNN
+F 3 "" H 1900 3550 50  0001 C CNN
+	1    1900 3550
+	0    1    1    0
+$EndComp
+Wire Wire Line
+	2050 3500 2050 3550
+Wire Wire Line
+	2000 3550 2150 3550
+Connection ~ 2050 3550
+$Comp
+L GND #PWR026
+U 1 1 5A78955B
+P 1800 3550
+F 0 "#PWR026" H 1800 3300 50  0001 C CNN
+F 1 "GND" H 1800 3400 50  0000 C CNN
+F 2 "" H 1800 3550 50  0001 C CNN
+F 3 "" H 1800 3550 50  0001 C CNN
+	1    1800 3550
+	0    1    1    0
+$EndComp
+Text GLabel 4700 3400 0    60   Input ~ 0
+XL1
+Text GLabel 4700 3500 0    60   Input ~ 0
+XL2
+$Comp
+L GND #PWR027
+U 1 1 5A78A3C0
+P 2750 3550
+F 0 "#PWR027" H 2750 3300 50  0001 C CNN
+F 1 "GND" H 2750 3400 50  0000 C CNN
+F 2 "" H 2750 3550 50  0001 C CNN
+F 3 "" H 2750 3550 50  0001 C CNN
+	1    2750 3550
+	0    -1   -1   0
+$EndComp
+$Comp
+L Conn_Coaxial J4
+U 1 1 5A78AAFF
+P 6950 1530
+F 0 "J4" H 6960 1650 50  0000 C CNN
+F 1 "Conn_Coaxial" V 7065 1530 50  0000 C CNN
+F 2 "Connectors:SMA_SMD_Jack_Straight" H 6950 1530 50  0001 C CNN
+F 3 "" H 6950 1530 50  0001 C CNN
+	1    6950 1530
+	-1   0    0    1
+$EndComp
+$Comp
+L GND #PWR028
+U 1 1 5A78B589
+P 6950 1330
+F 0 "#PWR028" H 6950 1080 50  0001 C CNN
+F 1 "GND" H 6950 1180 50  0000 C CNN
+F 2 "" H 6950 1330 50  0001 C CNN
+F 3 "" H 6950 1330 50  0001 C CNN
+	1    6950 1330
+	-1   0    0    1
+$EndComp
+Text GLabel 4700 4200 0    60   Input ~ 0
+ANEOMETER
 $EndSCHEMATC
