File: power.sch (KiCad schematic (older format))
At the start: 16 parts, among them U1 LT1129CS8-3.3, U4 LP3947

Commit message: basing solar power supply off of openMPPT
Parts:
- removed C19: C_Small, Capacitors_SMD:C_0603, symbol C_Small
- removed C27: C_Small, Capacitors_SMD:C_0402, symbol C_Small
- removed D3, D4: LED, LEDs:LED_0603_HandSoldering, symbol LED
- removed R14, R15, R19, R20: R_Small, Resistors_SMD:R_0603, symbol R_Small
- removed SC1: Solar_Cell, Connectors:PINHEAD1-2, symbol Solar_Cell
- removed U4: LP3947, Housings_SON:WSON-14_1EP_4.0x4.0mm_Pitch0.5mm, symbol LP3947
- added C19: -, Capacitors_SMD:C_0805, symbol C
- added C27, C32, C34, C37, C39: 1.0uF, Capacitors_SMD:C_0805, symbol C
- added C31, C33, C38, C41, C42: 0.1uF, Capacitors_SMD:C_0805, symbol C
- added C35, C36, C40, C43: CP, Capacitors_SMD:CP_Elec_6.3x7.7, symbol CP
- added D3: MBRD10100CT, TO_SOT_Packages_SMD:TO-252-2_Rectifier, symbol D_Schottky_x2_KCom_AKA
- added D4: D_Schottky, Diodes_SMD:D_SOD-523, symbol D_Schottky
- added D5, D6: LED, LEDs:LED_0805, symbol LED
- added J5: THERM, Connectors_Terminal_Blocks:TerminalBlock_Pheonix_MPT-2.54mm_2pol, symbol CONN_01X02
- added J6: SOLAR, Pin_Headers:Pin_Header_Straight_1x02_Pitch2.54mm, symbol CONN_01X02
- added L5: 3.3uH, Inductors:Inductor_Wurth_HCI-1890, symbol L_Core_Ferrite
- added Q2, Q3, Q4, Q5: FDMS8050, TO_SOT_Packages_SMD:TDSON-8-1, symbol FDMS8050
- added R14: 10k, Resistors_SMD:R_0603, symbol R
- added R15, R25, R26: 5.23k, Resistors_SMD:R_0603, symbol R
- added R19: 30.1k, Resistors_SMD:R_0603, symbol R
- added R20, R29: 499k, Resistors_SMD:R_0603, symbol R
- added R22: 36k, Resistors_SMD:R_0603, symbol R
- added R23: -, Resistors_SMD:R_0603, symbol R
- added R24: 10, Resistors_SMD:R_0603, symbol R
- added R27, R28: 0.010, Resistors_SMD:R_2512, symbol R
- added R30: 100k, Resistors_SMD:R_0603, symbol R
- added U4: BQ24650, Housings_DFN_QFN:QFN-16-1EP_3x3mm_Pitch0.5mm, symbol BQ24650
- C28: value C -> 1.0uF; footprint Capacitors_SMD:C_1206 -> Capacitors_SMD:C_0805; bom_partno (none) -> CL10A105KB8NNNC
Connections:
- net labels added: HIGH_DRIVE, LOW_DRIVE, MPPTSET, STAT1, STAT2, VREF
- net labels removed: SCL, SDA
- wire segments 25 -> 87
Other:
- note added: "Inductor must be rated >9A"
- note added: "Termination Enabled\nFor Lithium Batteries"
- moved on the sheet: BT1, BT2, BT3, BT4, U1

Commit message: i think that's enough for now
Parts:
- removed J5: THERM, Connectors_Terminal_Blocks:TerminalBlock_Pheonix_MPT-2.54mm_2pol, symbol CONN_01X02
- added TH1: Thermistor_NTC, Resistors_SMD:R_0805, symbol Thermistor_NTC
- C35, C43: value CP -> 100uF
- C36, C40: value CP -> 47uF
- R14: value 10k -> 10kΩ
- R15, R25, R26: value 5.23k -> 5.23kΩ
- R19: value 30.1k -> 30.1kΩ
- R20, R29: value 499k -> 499kΩ
- R22: value 36k -> 36kΩ
- R24: value 10 -> 10Ω
- R27, R28: value 0.010 -> 0.010Ω
- R30: value 100k -> 100kΩ
Connections:
- net GND: now also TH1.2
- net at C19.1, R14.1, R15.2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: now also TH1.1

Commit message: some cost savings
Parts:
- removed U1: LT1129CS8-3.3, Power_Integrations:SO-8C, symbol LT1129CS8-3.3
- added U1: LM1117-3.3, TO_SOT_Packages_SMD:SOT-223-3Lead_TabPin2, symbol LM1117-3.3
- added U6: LP3947, Housings_SON:WSON-14_1EP_4.0x4.0mm_Pitch0.5mm, symbol LP3947
Connections:
- net +3V3: now also U1.2 (VO)
- net GND: now also U1.1 (GND)
- net VCC: now also U1.3 (VI)
Changed lines of the file:
@@
 LIBS:sensors
 LIBS:SFUSat-power
+LIBS:battery_management
 LIBS:weather_station-cache
 EELAYER 25 0
@@
 $EndDescr
 $Comp
-L LT1129CS8-3.3 U1
-U 1 1 5A77DFCC
-P 6100 6000
-F 0 "U1" H 5750 6200 50  0000 C CNN
-F 1 "LT1129CS8-3.3" H 6300 6200 50  0000 C CNN
-F 2 "Power_Integrations:SO-8C" H 6100 6100 50  0000 C CIN
-F 3 "" H 6100 6000 50  0000 C CNN
-	1    6100 6000
-	1    0    0    -1
-$EndComp
-$Comp
-L +3.3V #PWR052
-U 1 1 5A77DFD3
-P 6715 6030
-F 0 "#PWR052" H 6715 5880 50  0001 C CNN
-F 1 "+3.3V" H 6715 6170 50  0000 C CNN
-F 2 "" H 6715 6030 50  0000 C CNN
-F 3 "" H 6715 6030 50  0000 C CNN
-	1    6715 6030
-	0    1    1    0
-$EndComp
-$Comp
-L GND #PWR053
-U 1 1 5A77DFD9
-P 6100 6450
-F 0 "#PWR053" H 6100 6200 50  0001 C CNN
-F 1 "GND" H 6100 6300 50  0000 C CNN
-F 2 "" H 6100 6450 50  0000 C CNN
-F 3 "" H 6100 6450 50  0000 C CNN
-	1    6100 6450
-	1    0    0    -1
-$EndComp
-$Comp
-L VCC #PWR054
-U 1 1 5A77DFDF
-P 5550 5950
-F 0 "#PWR054" H 5550 5800 50  0001 C CNN
-F 1 "VCC" H 5550 6100 50  0000 C CNN
-F 2 "" H 5550 5950 50  0000 C CNN
-F 3 "" H 5550 5950 50  0000 C CNN
-	1    5550 5950
-	0    -1   -1   0
-$EndComp
-Wire Wire Line
-	6000 6300 6000 6350
-Wire Wire Line
-	6000 6350 6200 6350
-Wire Wire Line
-	6100 6300 6100 6450
-Wire Wire Line
-	6200 6350 6200 6300
-Connection ~ 6100 6350
-Wire Wire Line
-	6650 5950 6710 5950
-Wire Wire Line
-	6710 5950 6710 6100
-Wire Wire Line
-	6710 6030 6715 6030
-Wire Wire Line
-	6710 6100 6650 6100
-Connection ~ 6710 6030
-$Comp
 L Battery_Cell BT1
 U 1 1 5A77DFF2
@@
 $EndComp
 $Comp
-L VCC #PWR055
+L VCC #PWR053
 U 1 1 5A77DFF9
 P 2150 5450
-F 0 "#PWR055" H 2150 5300 50  0001 C CNN
+F 0 "#PWR053" H 2150 5300 50  0001 C CNN
 F 1 "VCC" H 2150 5600 50  0000 C CNN
 F 2 "" H 2150 5450 50  0000 C CNN
@@
 $EndComp
 $Comp
-L GND #PWR056
+L GND #PWR054
 U 1 1 5A77DFFF
 P 2150 5750
-F 0 "#PWR056" H 2150 5500 50  0001 C CNN
+F 0 "#PWR054" H 2150 5500 50  0001 C CNN
 F 1 "GND" H 2150 5600 50  0000 C CNN
 F 2 "" H 2150 5750 50  0001 C CNN
@@
 $EndComp
 $Comp
-L VCC #PWR057
+L VCC #PWR055
 U 1 1 5A77E00C
 P 2800 5450
-F 0 "#PWR057" H 2800 5300 50  0001 C CNN
+F 0 "#PWR055" H 2800 5300 50  0001 C CNN
 F 1 "VCC" H 2800 5600 50  0000 C CNN
 F 2 "" H 2800 5450 50  0000 C CNN
@@
 $EndComp
 $Comp
-L GND #PWR058
+L GND #PWR056
 U 1 1 5A77E012
 P 2800 5750
-F 0 "#PWR058" H 2800 5500 50  0001 C CNN
+F 0 "#PWR056" H 2800 5500 50  0001 C CNN
 F 1 "GND" H 2800 5600 50  0000 C CNN
 F 2 "" H 2800 5750 50  0001 C CNN
@@
 $EndComp
 $Comp
-L VCC #PWR059
+L VCC #PWR057
 U 1 1 5A77E01F
 P 2150 5900
-F 0 "#PWR059" H 2150 5750 50  0001 C CNN
+F 0 "#PWR057" H 2150 5750 50  0001 C CNN
 F 1 "VCC" H 2150 6050 50  0000 C CNN
 F 2 "" H 2150 5900 50  0000 C CNN
@@
 $EndComp
 $Comp
-L GND #PWR060
+L GND #PWR058
 U 1 1 5A77E025
 P 2150 6200
-F 0 "#PWR060" H 2150 5950 50  0001 C CNN
+F 0 "#PWR058" H 2150 5950 50  0001 C CNN
 F 1 "GND" H 2150 6050 50  0000 C CNN
 F 2 "" H 2150 6200 50  0001 C CNN
@@
 $EndComp
 $Comp
-L VCC #PWR061
+L VCC #PWR059
 U 1 1 5A77E032
 P 2800 5900
-F 0 "#PWR061" H 2800 5750 50  0001 C CNN
+F 0 "#PWR059" H 2800 5750 50  0001 C CNN
 F 1 "VCC" H 2800 6050 50  0000 C CNN
 F 2 "" H 2800 5900 50  0000 C CNN
@@
 $EndComp
 $Comp
-L GND #PWR062
+L GND #PWR060
 U 1 1 5A77E038
 P 2800 6200
-F 0 "#PWR062" H 2800 5950 50  0001 C CNN
+F 0 "#PWR060" H 2800 5950 50  0001 C CNN
 F 1 "GND" H 2800 6050 50  0000 C CNN
 F 2 "" H 2800 6200 50  0001 C CNN
@@
 $EndComp
 $Comp
-L GND #PWR063
+L GND #PWR061
 U 1 1 5A773C84
 P 2600 1800
-F 0 "#PWR063" H 2600 1550 50  0001 C CNN
+F 0 "#PWR061" H 2600 1550 50  0001 C CNN
 F 1 "GND" H 2600 1650 50  0000 C CNN
 F 2 "" H 2600 1800 50  0001 C CNN
@@
 $EndComp
 $Comp
-L GND #PWR064
+L GND #PWR062
 U 1 1 5A773C88
 P 3800 2600
-F 0 "#PWR064" H 3800 2350 50  0001 C CNN
+F 0 "#PWR062" H 3800 2350 50  0001 C CNN
 F 1 "GND" H 3800 2450 50  0000 C CNN
 F 2 "" H 3800 2600 50  0001 C CNN
@@
 $EndComp
 $Comp
-L GND #PWR065
+L GND #PWR063
 U 1 1 5A773C8D
 P 3050 3850
-F 0 "#PWR065" H 3050 3600 50  0001 C CNN
+F 0 "#PWR063" H 3050 3600 50  0001 C CNN
 F 1 "GND" H 3050 3700 50  0000 C CNN
 F 2 "" H 3050 3850 50  0001 C CNN
@@
 $EndComp
 $Comp
-L GND #PWR066
+L GND #PWR064
 U 1 1 5A773C92
 P 2100 3900
-F 0 "#PWR066" H 2100 3650 50  0001 C CNN
+F 0 "#PWR064" H 2100 3650 50  0001 C CNN
 F 1 "GND" H 2100 3750 50  0000 C CNN
 F 2 "" H 2100 3900 50  0001 C CNN
@@
 $EndComp
 $Comp
-L GND #PWR067
+L GND #PWR065
 U 1 1 5A773C93
 P 1750 3900
-F 0 "#PWR067" H 1750 3650 50  0001 C CNN
+F 0 "#PWR065" H 1750 3650 50  0001 C CNN
 F 1 "GND" H 1750 3750 50  0000 C CNN
 F 2 "" H 1750 3900 50  0001 C CNN
@@
 $EndComp
 $Comp
-L GND #PWR068
+L GND #PWR066
 U 1 1 5A773C94
 P 1250 3850
-F 0 "#PWR068" H 1250 3600 50  0001 C CNN
+F 0 "#PWR066" H 1250 3600 50  0001 C CNN
 F 1 "GND" H 1250 3700 50  0000 C CNN
 F 2 "" H 1250 3850 50  0001 C CNN
@@
 VREF
 $Comp
-L GND #PWR069
+L GND #PWR067
 U 1 1 5A773C96
 P 4700 5050
-F 0 "#PWR069" H 4700 4800 50  0001 C CNN
+F 0 "#PWR067" H 4700 4800 50  0001 C CNN
 F 1 "GND" H 4700 4900 50  0000 C CNN
 F 2 "" H 4700 5050 50  0001 C CNN
@@
 $EndComp
 $Comp
-L GND #PWR070
+L GND #PWR068
 U 1 1 5A773C99
 P 5850 3750
-F 0 "#PWR070" H 5850 3500 50  0001 C CNN
+F 0 "#PWR068" H 5850 3500 50  0001 C CNN
 F 1 "GND" H 5850 3600 50  0000 C CNN
 F 2 "" H 5850 3750 50  0001 C CNN
@@
 $EndComp
 $Comp
-L GND #PWR071
+L GND #PWR069
 U 1 1 5A773C9E
 P 7050 3650
-F 0 "#PWR071" H 7050 3400 50  0001 C CNN
+F 0 "#PWR069" H 7050 3400 50  0001 C CNN
 F 1 "GND" H 7050 3500 50  0000 C CNN
 F 2 "" H 7050 3650 50  0001 C CNN
@@
 $EndComp
 $Comp
-L GND #PWR072
+L GND #PWR070
 U 1 1 5A773CA1
 P 7450 1300
-F 0 "#PWR072" H 7450 1050 50  0001 C CNN
+F 0 "#PWR070" H 7450 1050 50  0001 C CNN
 F 1 "GND" H 7450 1150 50  0000 C CNN
 F 2 "" H 7450 1300 50  0001 C CNN
@@
 $EndComp
 $Comp
-L GND #PWR073
+L GND #PWR071
 U 1 1 5A773CA4
 P 9200 3050
-F 0 "#PWR073" H 9200 2800 50  0001 C CNN
+F 0 "#PWR071" H 9200 2800 50  0001 C CNN
 F 1 "GND" H 9200 2900 50  0000 C CNN
 F 2 "" H 9200 3050 50  0001 C CNN
@@
 $EndComp
 $Comp
-L GND #PWR074
+L GND #PWR072
 U 1 1 5A773CA5
 P 7150 1300
-F 0 "#PWR074" H 7150 1050 50  0001 C CNN
+F 0 "#PWR072" H 7150 1050 50  0001 C CNN
 F 1 "GND" H 7150 1150 50  0000 C CNN
 F 2 "" H 7150 1300 50  0001 C CNN
@@
 $EndComp
 $Comp
-L GND #PWR075
+L GND #PWR073
 U 1 1 5A773CA8
 P 9800 4100
-F 0 "#PWR075" H 9800 3850 50  0001 C CNN
+F 0 "#PWR073" H 9800 3850 50  0001 C CNN
 F 1 "GND" H 9800 3950 50  0000 C CNN
 F 2 "" H 9800 4100 50  0001 C CNN
@@
 $EndComp
 $Comp
-L GND #PWR076
+L GND #PWR074
 U 1 1 5A773CB1
 P 7650 3650
-F 0 "#PWR076" H 7650 3400 50  0001 C CNN
+F 0 "#PWR074" H 7650 3400 50  0001 C CNN
 F 1 "GND" H 7650 3500 50  0000 C CNN
 F 2 "" H 7650 3650 50  0001 C CNN
@@
 $EndComp
 $Comp
-L GND #PWR077
+L GND #PWR075
 U 1 1 5A773CB3
 P 9450 3050
-F 0 "#PWR077" H 9450 2800 50  0001 C CNN
+F 0 "#PWR075" H 9450 2800 50  0001 C CNN
 F 1 "GND" H 9450 2900 50  0000 C CNN
 F 2 "" H 9450 3050 50  0001 C CNN
@@
 $EndComp
 $Comp
-L GND #PWR078
+L GND #PWR076
 U 1 1 5A773CB7
 P 7750 1300
-F 0 "#PWR078" H 7750 1050 50  0001 C CNN
+F 0 "#PWR076" H 7750 1050 50  0001 C CNN
 F 1 "GND" H 7750 1150 50  0000 C CNN
 F 2 "" H 7750 1300 50  0001 C CNN
@@
 $EndComp
 $Comp
-L GND #PWR079
+L GND #PWR077
 U 1 1 5A773CB9
 P 8050 1300
-F 0 "#PWR079" H 8050 1050 50  0001 C CNN
+F 0 "#PWR077" H 8050 1050 50  0001 C CNN
 F 1 "GND" H 8050 1150 50  0000 C CNN
 F 2 "" H 8050 1300 50  0001 C CNN
@@
 $EndComp
 $Comp
-L GND #PWR080
+L GND #PWR078
 U 1 1 5A773CBB
 P 9650 3050
-F 0 "#PWR080" H 9650 2800 50  0001 C CNN
+F 0 "#PWR078" H 9650 2800 50  0001 C CNN
 F 1 "GND" H 9650 2900 50  0000 C CNN
 F 2 "" H 9650 3050 50  0001 C CNN
@@
 Connection ~ 2750 1600
 $Comp
-L GND #PWR081
+L GND #PWR079
 U 1 1 5A773CBE
 P 2750 2650
-F 0 "#PWR081" H 2750 2400 50  0001 C CNN
+F 0 "#PWR079" H 2750 2400 50  0001 C CNN
 F 1 "GND" H 2750 2500 50  0000 C CNN
 F 2 "" H 2750 2650 50  0001 C CNN
@@
 	9000 2750 10100 2750
 $Comp
-L VCC #PWR082
+L VCC #PWR080
 U 1 1 5A77E21E
 P 10100 2750
-F 0 "#PWR082" H 10100 2600 50  0001 C CNN
+F 0 "#PWR080" H 10100 2600 50  0001 C CNN
 F 1 "VCC" H 10100 2900 50  0000 C CNN
 F 2 "" H 10100 2750 50  0001 C CNN
@@
 	1    0    0    -1
 $EndComp
+$Comp
+L VCC #PWR081
+U 1 1 5A77DFDF
+P 5800 5800
+F 0 "#PWR081" H 5800 5650 50  0001 C CNN
+F 1 "VCC" H 5800 5950 50  0000 C CNN
+F 2 "" H 5800 5800 50  0000 C CNN
+F 3 "" H 5800 5800 50  0000 C CNN
+	1    5800 5800
+	0    -1   -1   0
+$EndComp
+$Comp
+L LM1117-3.3 U1
+U 1 1 5A793E17
+P 6100 5800
+F 0 "U1" H 5950 5925 50  0000 C CNN
+F 1 "LM1117-3.3" H 6100 5925 50  0000 L CNN
+F 2 "TO_SOT_Packages_SMD:SOT-223-3Lead_TabPin2" H 6100 5800 50  0001 C CNN
+F 3 "" H 6100 5800 50  0001 C CNN
+	1    6100 5800
+	1    0    0    -1
+$EndComp
+$Comp
+L +3.3V #PWR082
+U 1 1 5A79439C
+P 6400 5800
+F 0 "#PWR082" H 6400 5650 50  0001 C CNN
+F 1 "+3.3V" H 6400 5940 50  0000 C CNN
+F 2 "" H 6400 5800 50  0001 C CNN
+F 3 "" H 6400 5800 50  0001 C CNN
+	1    6400 5800
+	0    1    1    0
+$EndComp
+$Comp
+L GND #PWR083
+U 1 1 5A79443A
+P 6100 6100
+F 0 "#PWR083" H 6100 5850 50  0001 C CNN
+F 1 "GND" H 6100 5950 50  0000 C CNN
+F 2 "" H 6100 6100 50  0001 C CNN
+F 3 "" H 6100 6100 50  0001 C CNN
+	1    6100 6100
+	1    0    0    -1
+$EndComp
+$Comp
+L LP3947 U6
+U 1 1 5A795B17
+P 10150 5400
+F 0 "U6" H 9650 6100 50  0000 L CNN
+F 1 "LP3947" H 9650 6000 50  0000 L CNN
+F 2 "Housings_SON:WSON-14_1EP_4.0x4.0mm_Pitch0.5mm" H 11350 4750 50  0001 C CNN
+F 3 "" H 10050 5600 50  0001 C CNN
+	1    10150 5400
+	1    0    0    -1
+$EndComp

Commit message: some changes
Parts:
- removed U1: LM1117-3.3, TO_SOT_Packages_SMD:SOT-223-3Lead_TabPin2, symbol LM1117-3.3
- removed U6: LP3947, Housings_SON:WSON-14_1EP_4.0x4.0mm_Pitch0.5mm, symbol LP3947
- added U1: LT1129-3.3_SOT223, TO_SOT_Packages_SMD:SOT-223-3Lead_TabPin2, symbol LT1129-3.3_SOT223
Connections:
- net +3V3: now also U1.3 (VO)
- net GND: now also U1.2 (GND)
- net VCC: now also U1.1 (VI)
Changed lines of the file:
@@
 $Descr A4 11693 8268
 encoding utf-8
-Sheet 3 4
+Sheet 3 3
 Title "OpenMPPT"
 Date "2017-07-08"
@@
 $EndComp
 $Comp
-L VCC #PWR053
+L VCC #PWR044
 U 1 1 5A77DFF9
 P 2150 5450
-F 0 "#PWR053" H 2150 5300 50  0001 C CNN
+F 0 "#PWR044" H 2150 5300 50  0001 C CNN
 F 1 "VCC" H 2150 5600 50  0000 C CNN
 F 2 "" H 2150 5450 50  0000 C CNN
@@
 $EndComp
 $Comp
-L GND #PWR054
+L GND #PWR045
 U 1 1 5A77DFFF
 P 2150 5750
-F 0 "#PWR054" H 2150 5500 50  0001 C CNN
+F 0 "#PWR045" H 2150 5500 50  0001 C CNN
 F 1 "GND" H 2150 5600 50  0000 C CNN
 F 2 "" H 2150 5750 50  0001 C CNN
@@
 $EndComp
 $Comp
-L VCC #PWR055
+L VCC #PWR046
 U 1 1 5A77E00C
 P 2800 5450
-F 0 "#PWR055" H 2800 5300 50  0001 C CNN
+F 0 "#PWR046" H 2800 5300 50  0001 C CNN
 F 1 "VCC" H 2800 5600 50  0000 C CNN
 F 2 "" H 2800 5450 50  0000 C CNN
@@
 $EndComp
 $Comp
-L GND #PWR056
+L GND #PWR047
 U 1 1 5A77E012
 P 2800 5750
-F 0 "#PWR056" H 2800 5500 50  0001 C CNN
+F 0 "#PWR047" H 2800 5500 50  0001 C CNN
 F 1 "GND" H 2800 5600 50  0000 C CNN
 F 2 "" H 2800 5750 50  0001 C CNN
@@
 $EndComp
 $Comp
-L VCC #PWR057
+L VCC #PWR048
 U 1 1 5A77E01F
 P 2150 5900
-F 0 "#PWR057" H 2150 5750 50  0001 C CNN
+F 0 "#PWR048" H 2150 5750 50  0001 C CNN
 F 1 "VCC" H 2150 6050 50  0000 C CNN
 F 2 "" H 2150 5900 50  0000 C CNN
@@
 $EndComp
 $Comp
-L GND #PWR058
+L GND #PWR049
 U 1 1 5A77E025
 P 2150 6200
-F 0 "#PWR058" H 2150 5950 50  0001 C CNN
+F 0 "#PWR049" H 2150 5950 50  0001 C CNN
 F 1 "GND" H 2150 6050 50  0000 C CNN
 F 2 "" H 2150 6200 50  0001 C CNN
@@
 $EndComp
 $Comp
-L VCC #PWR059
+L VCC #PWR050
 U 1 1 5A77E032
 P 2800 5900
-F 0 "#PWR059" H 2800 5750 50  0001 C CNN
+F 0 "#PWR050" H 2800 5750 50  0001 C CNN
 F 1 "VCC" H 2800 6050 50  0000 C CNN
 F 2 "" H 2800 5900 50  0000 C CNN
@@
 $EndComp
 $Comp
-L GND #PWR060
+L GND #PWR051
 U 1 1 5A77E038
 P 2800 6200
-F 0 "#PWR060" H 2800 5950 50  0001 C CNN
+F 0 "#PWR051" H 2800 5950 50  0001 C CNN
 F 1 "GND" H 2800 6050 50  0000 C CNN
 F 2 "" H 2800 6200 50  0001 C CNN
@@
 $EndComp
 $Comp
-L GND #PWR061
+L GND #PWR052
 U 1 1 5A773C84
 P 2600 1800
-F 0 "#PWR061" H 2600 1550 50  0001 C CNN
+F 0 "#PWR052" H 2600 1550 50  0001 C CNN
 F 1 "GND" H 2600 1650 50  0000 C CNN
 F 2 "" H 2600 1800 50  0001 C CNN
@@
 $EndComp
 $Comp
-L GND #PWR062
+L GND #PWR053
 U 1 1 5A773C88
 P 3800 2600
-F 0 "#PWR062" H 3800 2350 50  0001 C CNN
+F 0 "#PWR053" H 3800 2350 50  0001 C CNN
 F 1 "GND" H 3800 2450 50  0000 C CNN
 F 2 "" H 3800 2600 50  0001 C CNN
@@
 $EndComp
 $Comp
-L GND #PWR063
+L GND #PWR054
 U 1 1 5A773C8D
 P 3050 3850
-F 0 "#PWR063" H 3050 3600 50  0001 C CNN
+F 0 "#PWR054" H 3050 3600 50  0001 C CNN
 F 1 "GND" H 3050 3700 50  0000 C CNN
 F 2 "" H 3050 3850 50  0001 C CNN
@@
 $EndComp
 $Comp
-L GND #PWR064
+L GND #PWR055
 U 1 1 5A773C92
 P 2100 3900
-F 0 "#PWR064" H 2100 3650 50  0001 C CNN
+F 0 "#PWR055" H 2100 3650 50  0001 C CNN
 F 1 "GND" H 2100 3750 50  0000 C CNN
 F 2 "" H 2100 3900 50  0001 C CNN
@@
 $EndComp
 $Comp
-L GND #PWR065
+L GND #PWR056
 U 1 1 5A773C93
 P 1750 3900
-F 0 "#PWR065" H 1750 3650 50  0001 C CNN
+F 0 "#PWR056" H 1750 3650 50  0001 C CNN
 F 1 "GND" H 1750 3750 50  0000 C CNN
 F 2 "" H 1750 3900 50  0001 C CNN
@@
 $EndComp
 $Comp
-L GND #PWR066
+L GND #PWR057
 U 1 1 5A773C94
 P 1250 3850
-F 0 "#PWR066" H 1250 3600 50  0001 C CNN
+F 0 "#PWR057" H 1250 3600 50  0001 C CNN
 F 1 "GND" H 1250 3700 50  0000 C CNN
 F 2 "" H 1250 3850 50  0001 C CNN
@@
 VREF
 $Comp
-L GND #PWR067
+L GND #PWR058
 U 1 1 5A773C96
 P 4700 5050
-F 0 "#PWR067" H 4700 4800 50  0001 C CNN
+F 0 "#PWR058" H 4700 4800 50  0001 C CNN
 F 1 "GND" H 4700 4900 50  0000 C CNN
 F 2 "" H 4700 5050 50  0001 C CNN
@@
 $EndComp
 $Comp
-L GND #PWR068
+L GND #PWR059
 U 1 1 5A773C99
 P 5850 3750
-F 0 "#PWR068" H 5850 3500 50  0001 C CNN
+F 0 "#PWR059" H 5850 3500 50  0001 C CNN
 F 1 "GND" H 5850 3600 50  0000 C CNN
 F 2 "" H 5850 3750 50  0001 C CNN
@@
 $EndComp
 $Comp
-L GND #PWR069
+L GND #PWR060
 U 1 1 5A773C9E
 P 7050 3650
-F 0 "#PWR069" H 7050 3400 50  0001 C CNN
+F 0 "#PWR060" H 7050 3400 50  0001 C CNN
 F 1 "GND" H 7050 3500 50  0000 C CNN
 F 2 "" H 7050 3650 50  0001 C CNN
@@
 $EndComp
 $Comp
-L GND #PWR070
+L GND #PWR061
 U 1 1 5A773CA1
 P 7450 1300
-F 0 "#PWR070" H 7450 1050 50  0001 C CNN
+F 0 "#PWR061" H 7450 1050 50  0001 C CNN
 F 1 "GND" H 7450 1150 50  0000 C CNN
 F 2 "" H 7450 1300 50  0001 C CNN
@@
 $EndComp
 $Comp
-L GND #PWR071
+L GND #PWR062
 U 1 1 5A773CA4
 P 9200 3050
-F 0 "#PWR071" H 9200 2800 50  0001 C CNN
+F 0 "#PWR062" H 9200 2800 50  0001 C CNN
 F 1 "GND" H 9200 2900 50  0000 C CNN
 F 2 "" H 9200 3050 50  0001 C CNN
@@
 $EndComp
 $Comp
-L GND #PWR072
+L GND #PWR063
 U 1 1 5A773CA5
 P 7150 1300
-F 0 "#PWR072" H 7150 1050 50  0001 C CNN
+F 0 "#PWR063" H 7150 1050 50  0001 C CNN
 F 1 "GND" H 7150 1150 50  0000 C CNN
 F 2 "" H 7150 1300 50  0001 C CNN
@@
 $EndComp
 $Comp
-L GND #PWR073
+L GND #PWR064
 U 1 1 5A773CA8
 P 9800 4100
-F 0 "#PWR073" H 9800 3850 50  0001 C CNN
+F 0 "#PWR064" H 9800 3850 50  0001 C CNN
 F 1 "GND" H 9800 3950 50  0000 C CNN
 F 2 "" H 9800 4100 50  0001 C CNN
@@
 $EndComp
 $Comp
-L GND #PWR074
+L GND #PWR065
 U 1 1 5A773CB1
 P 7650 3650
-F 0 "#PWR074" H 7650 3400 50  0001 C CNN
+F 0 "#PWR065" H 7650 3400 50  0001 C CNN
 F 1 "GND" H 7650 3500 50  0000 C CNN
 F 2 "" H 7650 3650 50  0001 C CNN
@@
 $EndComp
 $Comp
-L GND #PWR075
+L GND #PWR066
 U 1 1 5A773CB3
 P 9450 3050
-F 0 "#PWR075" H 9450 2800 50  0001 C CNN
+F 0 "#PWR066" H 9450 2800 50  0001 C CNN
 F 1 "GND" H 9450 2900 50  0000 C CNN
 F 2 "" H 9450 3050 50  0001 C CNN
@@
 $EndComp
 $Comp
-L GND #PWR076
+L GND #PWR067
 U 1 1 5A773CB7
 P 7750 1300
-F 0 "#PWR076" H 7750 1050 50  0001 C CNN
+F 0 "#PWR067" H 7750 1050 50  0001 C CNN
 F 1 "GND" H 7750 1150 50  0000 C CNN
 F 2 "" H 7750 1300 50  0001 C CNN
@@
 $EndComp
 $Comp
-L GND #PWR077
+L GND #PWR068
 U 1 1 5A773CB9
 P 8050 1300
-F 0 "#PWR077" H 8050 1050 50  0001 C CNN
+F 0 "#PWR068" H 8050 1050 50  0001 C CNN
 F 1 "GND" H 8050 1150 50  0000 C CNN
 F 2 "" H 8050 1300 50  0001 C CNN
@@
 $EndComp
 $Comp
-L GND #PWR078
+L GND #PWR069
 U 1 1 5A773CBB
 P 9650 3050
-F 0 "#PWR078" H 9650 2800 50  0001 C CNN
+F 0 "#PWR069" H 9650 2800 50  0001 C CNN
 F 1 "GND" H 9650 2900 50  0000 C CNN
 F 2 "" H 9650 3050 50  0001 C CNN
@@
 Connection ~ 2750 1600
 $Comp
-L GND #PWR079
+L GND #PWR070
 U 1 1 5A773CBE
 P 2750 2650
-F 0 "#PWR079" H 2750 2400 50  0001 C CNN
+F 0 "#PWR070" H 2750 2400 50  0001 C CNN
 F 1 "GND" H 2750 2500 50  0000 C CNN
 F 2 "" H 2750 2650 50  0001 C CNN
@@
 	9000 2750 10100 2750
 $Comp
-L VCC #PWR080
+L VCC #PWR071
 U 1 1 5A77E21E
 P 10100 2750
-F 0 "#PWR080" H 10100 2600 50  0001 C CNN
+F 0 "#PWR071" H 10100 2600 50  0001 C CNN
 F 1 "VCC" H 10100 2900 50  0000 C CNN
 F 2 "" H 10100 2750 50  0001 C CNN
@@
 $EndComp
 $Comp
-L VCC #PWR081
+L VCC #PWR072
 U 1 1 5A77DFDF
 P 5800 5800
-F 0 "#PWR081" H 5800 5650 50  0001 C CNN
+F 0 "#PWR072" H 5800 5650 50  0001 C CNN
 F 1 "VCC" H 5800 5950 50  0000 C CNN
 F 2 "" H 5800 5800 50  0000 C CNN
@@
 $EndComp
 $Comp
-L LM1117-3.3 U1
-U 1 1 5A793E17
-P 6100 5800
-F 0 "U1" H 5950 5925 50  0000 C CNN
-F 1 "LM1117-3.3" H 6100 5925 50  0000 L CNN
-F 2 "TO_SOT_Packages_SMD:SOT-223-3Lead_TabPin2" H 6100 5800 50  0001 C CNN
-F 3 "" H 6100 5800 50  0001 C CNN
-	1    6100 5800
-	1    0    0    -1
-$EndComp
-$Comp
-L +3.3V #PWR082
+L +3.3V #PWR073
 U 1 1 5A79439C
 P 6400 5800
-F 0 "#PWR082" H 6400 5650 50  0001 C CNN
+F 0 "#PWR073" H 6400 5650 50  0001 C CNN
 F 1 "+3.3V" H 6400 5940 50  0000 C CNN
 F 2 "" H 6400 5800 50  0001 C CNN
@@
 $EndComp
 $Comp
-L GND #PWR083
+L GND #PWR074
 U 1 1 5A79443A
 P 6100 6100
-F 0 "#PWR083" H 6100 5850 50  0001 C CNN
+F 0 "#PWR074" H 6100 5850 50  0001 C CNN
 F 1 "GND" H 6100 5950 50  0000 C CNN
 F 2 "" H 6100 6100 50  0001 C CNN
@@
 $EndComp
 $Comp
-L LP3947 U6
-U 1 1 5A795B17
-P 10150 5400
-F 0 "U6" H 9650 6100 50  0000 L CNN
-F 1 "LP3947" H 9650 6000 50  0000 L CNN
-F 2 "Housings_SON:WSON-14_1EP_4.0x4.0mm_Pitch0.5mm" H 11350 4750 50  0001 C CNN
-F 3 "" H 10050 5600 50  0001 C CNN
-	1    10150 5400
-	1    0    0    -1
-$EndComp
+L LT1129-3.3_SOT223 U1
+U 1 1 5AC328C0
+P 6100 5800
+F 0 "U1" H 5950 5925 50  0000 C CNN
+F 1 "LT1129-3.3_SOT223" H 6100 5925 50  0000 L CNN
+F 2 "TO_SOT_Packages_SMD:SOT-223-3Lead_TabPin2" H 6100 6025 50  0001 C CIN
+F 3 "" H 6100 5750 50  0001 C CNN
+	1    6100 5800
+	1    0    0    -1
+$EndComp
