File: radio.sch (KiCad schematic (older format))
At the start: 10 parts, among them J3 Conn_Coaxial, Q1 Q_NMOS_DGS

Commit message: i think that's enough for now
Parts:
- R16: value 100K -> 100kΩ
- R17: value 3.3k -> 3.3kΩ
- R18: value 1.8K -> 1.8KΩ
Changed lines of the file:
@@
 P 4850 2400
 F 0 "R16" H 4880 2420 50  0000 L CNN
-F 1 "100K" H 4880 2360 50  0000 L CNN
+F 1 "100kΩ" H 4880 2360 50  0000 L CNN
 F 2 "Resistors_SMD:R_0603" H 4850 2400 50  0001 C CNN
 F 3 "" H 4850 2400 50  0001 C CNN
@@
 Connection ~ 4400 2400
 $Comp
-L GND #PWR43
+L GND #PWR041
 U 1 1 5A76777A
 P 4400 2050
-F 0 "#PWR43" H 4400 1800 50  0001 C CNN
+F 0 "#PWR041" H 4400 1800 50  0001 C CNN
 F 1 "GND" H 4400 1900 50  0000 C CNN
 F 2 "" H 4400 2050 50  0001 C CNN
@@
 $EndComp
 $Comp
-L GND #PWR41
+L GND #PWR042
 U 1 1 5A7677D4
 P 3450 2800
-F 0 "#PWR41" H 3450 2550 50  0001 C CNN
+F 0 "#PWR042" H 3450 2550 50  0001 C CNN
 F 1 "GND" H 3450 2650 50  0000 C CNN
 F 2 "" H 3450 2800 50  0001 C CNN
@@
 $EndComp
 $Comp
-L GND #PWR44
+L GND #PWR043
 U 1 1 5A767824
 P 5600 3250
-F 0 "#PWR44" H 5600 3000 50  0001 C CNN
+F 0 "#PWR043" H 5600 3000 50  0001 C CNN
 F 1 "GND" H 5600 3100 50  0000 C CNN
 F 2 "" H 5600 3250 50  0001 C CNN
@@
 $EndComp
 $Comp
-L GND #PWR45
+L GND #PWR044
 U 1 1 5A767847
 P 5700 3250
-F 0 "#PWR45" H 5700 3000 50  0001 C CNN
+F 0 "#PWR044" H 5700 3000 50  0001 C CNN
 F 1 "GND" H 5700 3100 50  0000 C CNN
 F 2 "" H 5700 3250 50  0001 C CNN
@@
 $EndComp
 $Comp
-L VCC #PWR46
+L VCC #PWR045
 U 1 1 5A76788D
 P 5800 3250
-F 0 "#PWR46" H 5800 3100 50  0001 C CNN
+F 0 "#PWR045" H 5800 3100 50  0001 C CNN
 F 1 "VCC" H 5800 3400 50  0000 C CNN
 F 2 "" H 5800 3250 50  0001 C CNN
@@
 	6800 2800 6250 2800
 $Comp
-L GND #PWR51
+L GND #PWR046
 U 1 1 5A767A36
 P 7200 2800
-F 0 "#PWR51" H 7200 2550 50  0001 C CNN
+F 0 "#PWR046" H 7200 2550 50  0001 C CNN
 F 1 "GND" H 7200 2650 50  0000 C CNN
 F 2 "" H 7200 2800 50  0001 C CNN
@@
 P 6450 4250
 F 0 "R17" H 6480 4270 50  0000 L CNN
-F 1 "3.3k" H 6480 4210 50  0000 L CNN
+F 1 "3.3kΩ" H 6480 4210 50  0000 L CNN
 F 2 "Resistors_SMD:R_0603" H 6450 4250 50  0001 C CNN
 F 3 "" H 6450 4250 50  0001 C CNN
@@
 P 6650 4450
 F 0 "R18" H 6680 4470 50  0000 L CNN
-F 1 "1.8K" H 6680 4410 50  0000 L CNN
+F 1 "1.8KΩ" H 6680 4410 50  0000 L CNN
 F 2 "Resistors_SMD:R_0603" H 6650 4450 50  0001 C CNN
 F 3 "" H 6650 4450 50  0001 C CNN
@@
 Connection ~ 6650 4250
 $Comp
-L GND #PWR50
+L GND #PWR047
 U 1 1 5A767DBD
 P 6350 4250
-F 0 "#PWR50" H 6350 4000 50  0001 C CNN
+F 0 "#PWR047" H 6350 4000 50  0001 C CNN
 F 1 "GND" H 6350 4100 50  0000 C CNN
 F 2 "" H 6350 4250 50  0001 C CNN
@@
 $EndComp
 $Comp
-L GND #PWR49
+L GND #PWR048
 U 1 1 5A768602
 P 6250 3600
-F 0 "#PWR49" H 6250 3350 50  0001 C CNN
+F 0 "#PWR048" H 6250 3350 50  0001 C CNN
 F 1 "GND" H 6250 3450 50  0000 C CNN
 F 2 "" H 6250 3600 50  0001 C CNN
@@
 $EndComp
 $Comp
-L GND #PWR48
+L GND #PWR049
 U 1 1 5A7686F2
 P 6250 2600
-F 0 "#PWR48" H 6250 2350 50  0001 C CNN
+F 0 "#PWR049" H 6250 2350 50  0001 C CNN
 F 1 "GND" H 6250 2450 50  0000 C CNN
 F 2 "" H 6250 2600 50  0001 C CNN
@@
 $EndComp
 $Comp
-L GND #PWR47
+L GND #PWR050
 U 1 1 5A76871A
 P 6250 2400
-F 0 "#PWR47" H 6250 2150 50  0001 C CNN
+F 0 "#PWR050" H 6250 2150 50  0001 C CNN
 F 1 "GND" H 6250 2250 50  0000 C CNN
 F 2 "" H 6250 2400 50  0001 C CNN
@@
 	3950 3000 3600 3000
 $Comp
-L GND #PWR42
+L GND #PWR051
 U 1 1 5A769BBF
 P 4150 3200
-F 0 "#PWR42" H 4150 2950 50  0001 C CNN
+F 0 "#PWR051" H 4150 2950 50  0001 C CNN
 F 1 "GND" H 4150 3050 50  0000 C CNN
 F 2 "" H 4150 3200 50  0001 C CNN
