File: sensors.sch (KiCad schematic (older format))
At the start: 27 parts, among them M1 ANEOMETER, U2 ADS1120-PW, U5 MPL115A1, U6 MPU-9250

Commit message: some cost savings
Parts:
- removed C24: 10nF, Capacitors_SMD:C_0402, symbol C_Small
- removed C25: 100nF, Capacitors_SMD:C_0402, symbol C_Small
- removed C26: C_Small, Capacitors_SMD:C_0402, symbol C_Small
- removed U6: MPU-9250, Housings_DFN_QFN:QFN-24-1EP_3x3mm_Pitch0.4mm, symbol MPU-9250
Changed lines of the file:
@@
 LIBS:sensors
 LIBS:SFUSat-power
+LIBS:battery_management
 LIBS:weather_station-cache
 EELAYER 25 0
@@
 SPI_MSI
 $Comp
-L GND #PWR083
+L GND #PWR084
 U 1 1 5A776C76
 P 4100 4100
-F 0 "#PWR083" H 4100 3850 50  0001 C CNN
+F 0 "#PWR084" H 4100 3850 50  0001 C CNN
 F 1 "GND" H 4100 3950 50  0000 C CNN
 F 2 "" H 4100 4100 50  0001 C CNN
@@
 $EndComp
 $Comp
-L +3.3V #PWR084
+L +3.3V #PWR085
 U 1 1 5A776C7C
 P 5300 4100
-F 0 "#PWR084" H 5300 3950 50  0001 C CNN
+F 0 "#PWR085" H 5300 3950 50  0001 C CNN
 F 1 "+3.3V" H 5300 4240 50  0000 C CNN
 F 2 "" H 5300 4100 50  0001 C CNN
@@
 $EndComp
 $Comp
-L GND #PWR085
+L GND #PWR086
 U 1 1 5A776C89
 P 4500 4600
-F 0 "#PWR085" H 4500 4350 50  0001 C CNN
+F 0 "#PWR086" H 4500 4350 50  0001 C CNN
 F 1 "GND" H 4500 4450 50  0000 C CNN
 F 2 "" H 4500 4600 50  0001 C CNN
@@
 $EndComp
 $Comp
-L GND #PWR086
+L GND #PWR087
 U 1 1 5A777E2B
 P 1400 2450
-F 0 "#PWR086" H 1400 2200 50  0001 C CNN
+F 0 "#PWR087" H 1400 2200 50  0001 C CNN
 F 1 "GND" H 1400 2300 50  0000 C CNN
 F 2 "" H 1400 2450 50  0000 C CNN
@@
 $EndComp
 $Comp
-L GND #PWR087
+L GND #PWR088
 U 1 1 5A777E31
 P 2100 2450
-F 0 "#PWR087" H 2100 2200 50  0001 C CNN
+F 0 "#PWR088" H 2100 2200 50  0001 C CNN
 F 1 "GND" H 2100 2300 50  0000 C CNN
 F 2 "" H 2100 2450 50  0000 C CNN
@@
 $EndComp
 $Comp
-L GND #PWR088
+L GND #PWR089
 U 1 1 5A777E37
 P 2050 1650
-F 0 "#PWR088" H 2050 1400 50  0001 C CNN
+F 0 "#PWR089" H 2050 1400 50  0001 C CNN
 F 1 "GND" H 2050 1500 50  0000 C CNN
 F 2 "" H 2050 1650 50  0000 C CNN
@@
 SPI_DRDY
 $Comp
-L +3.3V #PWR089
+L +3.3V #PWR090
 U 1 1 5A777E43
 P 2050 3450
-F 0 "#PWR089" H 2050 3300 50  0001 C CNN
+F 0 "#PWR090" H 2050 3300 50  0001 C CNN
 F 1 "+3.3V" H 2050 3590 50  0000 C CNN
 F 2 "" H 2050 3450 50  0000 C CNN
@@
 $EndComp
 $Comp
-L GND #PWR090
+L GND #PWR091
 U 1 1 5A777E49
 P 2050 4600
-F 0 "#PWR090" H 2050 4350 50  0001 C CNN
+F 0 "#PWR091" H 2050 4350 50  0001 C CNN
 F 1 "GND" H 2050 4450 50  0000 C CNN
 F 2 "" H 2050 4600 50  0000 C CNN
@@
 Connection ~ 2050 4600
 $Comp
-L +3.3V #PWR091
+L +3.3V #PWR092
 U 1 1 5A777E65
 P 1450 1650
-F 0 "#PWR091" H 1450 1500 50  0001 C CNN
+F 0 "#PWR092" H 1450 1500 50  0001 C CNN
 F 1 "+3.3V" H 1450 1790 50  0000 C CNN
 F 2 "" H 1450 1650 50  0000 C CNN
@@
 $EndComp
 $Comp
-L GND #PWR092
+L GND #PWR093
 U 1 1 5A777E9E
 P 2600 2450
-F 0 "#PWR092" H 2600 2200 50  0001 C CNN
+F 0 "#PWR093" H 2600 2200 50  0001 C CNN
 F 1 "GND" H 2600 2300 50  0000 C CNN
 F 2 "" H 2600 2450 50  0000 C CNN
@@
 $EndComp
 $Comp
-L GND #PWR093
+L GND #PWR094
 U 1 1 5A777EA4
 P 3300 2450
-F 0 "#PWR093" H 3300 2200 50  0001 C CNN
+F 0 "#PWR094" H 3300 2200 50  0001 C CNN
 F 1 "GND" H 3300 2300 50  0000 C CNN
 F 2 "" H 3300 2450 50  0000 C CNN
@@
 $EndComp
 $Comp
-L GND #PWR094
+L GND #PWR095
 U 1 1 5A777EAA
 P 3250 1650
-F 0 "#PWR094" H 3250 1400 50  0001 C CNN
+F 0 "#PWR095" H 3250 1400 50  0001 C CNN
 F 1 "GND" H 3250 1500 50  0000 C CNN
 F 2 "" H 3250 1650 50  0000 C CNN
@@
 Connection ~ 2850 1650
 $Comp
-L +3.3V #PWR095
+L +3.3V #PWR096
 U 1 1 5A777EBE
 P 2650 1650
-F 0 "#PWR095" H 2650 1500 50  0001 C CNN
+F 0 "#PWR096" H 2650 1500 50  0001 C CNN
 F 1 "+3.3V" H 2650 1790 50  0000 C CNN
 F 2 "" H 2650 1650 50  0000 C CNN
@@
 CS_ADS1120
 $Comp
-L +3.3V #PWR096
-U 1 1 5A778A93
-P 7350 2450
-F 0 "#PWR096" H 7350 2300 50  0001 C CNN
-F 1 "+3.3V" H 7350 2590 50  0000 C CNN
-F 2 "" H 7350 2450 50  0001 C CNN
-F 3 "" H 7350 2450 50  0001 C CNN
-	1    7350 2450
-	1    0    0    -1
-$EndComp
-$Comp
-L C_Small C25
-U 1 1 5A778C97
-P 7700 2700
-F 0 "C25" H 7710 2770 50  0000 L CNN
-F 1 "100nF" H 7300 2600 50  0000 L CNN
-F 2 "Capacitors_SMD:C_0402" H 7700 2700 50  0001 C CNN
-F 3 "" H 7700 2700 50  0001 C CNN
-	1    7700 2700
-	0    1    1    0
-$EndComp
-Wire Wire Line
-	7600 2700 7450 2700
-Wire Wire Line
-	7450 2450 7450 2800
-Connection ~ 7450 2700
-$Comp
-L GND #PWR097
-U 1 1 5A778EB0
-P 7800 2700
-F 0 "#PWR097" H 7800 2450 50  0001 C CNN
-F 1 "GND" H 7800 2550 50  0000 C CNN
-F 2 "" H 7800 2700 50  0001 C CNN
-F 3 "" H 7800 2700 50  0001 C CNN
-	1    7800 2700
-	0    -1   -1   0
-$EndComp
-$Comp
-L +3.3V #PWR098
-U 1 1 5A779442
-P 8050 4000
-F 0 "#PWR098" H 8050 3850 50  0001 C CNN
-F 1 "+3.3V" H 8050 4140 50  0000 C CNN
-F 2 "" H 8050 4000 50  0001 C CNN
-F 3 "" H 8050 4000 50  0001 C CNN
-	1    8050 4000
-	0    1    1    0
-$EndComp
-$Comp
-L GND #PWR099
-U 1 1 5A77947C
-P 8050 4100
-F 0 "#PWR099" H 8050 3850 50  0001 C CNN
-F 1 "GND" H 8050 3950 50  0000 C CNN
-F 2 "" H 8050 4100 50  0001 C CNN
-F 3 "" H 8050 4100 50  0001 C CNN
-	1    8050 4100
-	1    0    0    -1
-$EndComp
-$Comp
-L C_Small C26
-U 1 1 5A77960C
-P 8350 3900
-F 0 "C26" H 8360 3970 50  0000 L CNN
-F 1 "C_Small" H 8360 3820 50  0000 L CNN
-F 2 "Capacitors_SMD:C_0402" H 8350 3900 50  0001 C CNN
-F 3 "" H 8350 3900 50  0001 C CNN
-	1    8350 3900
-	0    1    1    0
-$EndComp
-Wire Wire Line
-	8050 3900 8250 3900
-$Comp
-L GND #PWR0100
-U 1 1 5A779778
-P 8450 3900
-F 0 "#PWR0100" H 8450 3650 50  0001 C CNN
-F 1 "GND" H 8450 3750 50  0000 C CNN
-F 2 "" H 8450 3900 50  0001 C CNN
-F 3 "" H 8450 3900 50  0001 C CNN
-	1    8450 3900
-	0    -1   -1   0
-$EndComp
-$Comp
-L GND #PWR0101
-U 1 1 5A77987C
-P 6650 3900
-F 0 "#PWR0101" H 6650 3650 50  0001 C CNN
-F 1 "GND" H 6650 3750 50  0000 C CNN
-F 2 "" H 6650 3900 50  0001 C CNN
-F 3 "" H 6650 3900 50  0001 C CNN
-	1    6650 3900
-	0    1    1    0
-$EndComp
-Text GLabel 8050 3400 2    60   Input ~ 0
-MPU_INT
-$Comp
-L C_Small C24
-U 1 1 5A779AEA
-P 7250 2700
-F 0 "C24" H 7260 2770 50  0000 L CNN
-F 1 "10nF" H 7260 2620 50  0000 L CNN
-F 2 "Capacitors_SMD:C_0402" H 7250 2700 50  0001 C CNN
-F 3 "" H 7250 2700 50  0001 C CNN
-	1    7250 2700
-	1    0    0    -1
-$EndComp
-Wire Wire Line
-	7250 2600 7250 2450
-Wire Wire Line
-	7250 2450 7450 2450
-Connection ~ 7350 2450
-$Comp
-L MPU-9250 U6
-U 1 1 5A77ADF0
-P 7350 3700
-F 0 "U6" H 6900 4450 50  0000 C CNN
-F 1 "MPU-9250" H 7650 2950 50  0000 C CNN
-F 2 "Housings_DFN_QFN:QFN-24-1EP_3x3mm_Pitch0.4mm" H 7350 2700 50  0001 C CNN
-F 3 "" H 7350 3550 50  0001 C CNN
-	1    7350 3700
-	1    0    0    -1
-$EndComp
-$Comp
-L GND #PWR0102
-U 1 1 5A77AEB3
-P 7350 4600
-F 0 "#PWR0102" H 7350 4350 50  0001 C CNN
-F 1 "GND" H 7350 4450 50  0000 C CNN
-F 2 "" H 7350 4600 50  0001 C CNN
-F 3 "" H 7350 4600 50  0001 C CNN
-	1    7350 4600
-	1    0    0    -1
-$EndComp
-$Comp
 L Mounting_Hole_PAD MK8
 U 1 1 5A77D205
@@
 	1    0    0    -1
 $EndComp
-Text GLabel 6650 3600 0    60   Input ~ 0
-SCL
-Text GLabel 6650 3400 0    60   Input ~ 0
-SDA
 $Comp
 L Fan M1
@@
 $EndComp
 $Comp
-L +3.3V #PWR0103
+L +3.3V #PWR097
 U 1 1 5A76B491
 P 4000 5500
-F 0 "#PWR0103" H 4000 5350 50  0001 C CNN
+F 0 "#PWR097" H 4000 5350 50  0001 C CNN
 F 1 "+3.3V" H 4000 5640 50  0000 C CNN
 F 2 "" H 4000 5500 50  0001 C CNN

Commit message: some changes
Parts:
- removed C16, C18, C5, C7: F_cap, Capacitors_SMD:C_0402, symbol C_Small
- removed C17, C6: Diff_Cap, Capacitors_SMD:C_0402, symbol C_Small
- removed C23: 1uF, Capacitors_SMD:C_0402, symbol C_Small
- removed MK5, MK6, MK7, MK8: Mounting_Hole_PAD, Measurement_Points:Measurement_Point_Square-SMD-Pad_Big, symbol Mounting_Hole_PAD
- removed R1, R10, R13, R6: 10MΩ, Resistors_SMD:R_0603, symbol R_Small
- removed R11, R12, R4, R5: 510Ω, Resistors_SMD:R_0603, symbol R_Small
- removed U2: ADS1120-PW, Housings_SSOP:TSSOP-16_4.4x5mm_Pitch0.65mm, symbol ADS1120-PW
- removed U5: MPL115A1, Housings_LGA:LGA-8_3x5mm_Pitch1.25mm, symbol MPL115A1
Other:
- moved on the sheet: M1, R21
