File: weather_station.kicad_pcb (KiCad board)
At the start: 2 copper layers, 100 x 140 mm, 117 parts, among them J2 Conn_02x10_Odd_Even, J3 Conn_Coaxial, J4 Conn_Coaxial, J6 SOLAR, M1 ANEOMETER, Q1 Q_NMOS_DGS, Q2 FDMS8050, Q3 FDMS8050, Q4 FDMS8050, Q5 FDMS8050, U1 LT1129CS8-3.3, U2 ADS1120-PW, U3 nRF52832, U4 BQ24650, U5 MPL115A1, U6 MPU-9250, Y1 FL3200037, Y2 32.786khz

Commit message: some cost savings
Parts:
- moved R28 0.73 mm to (37.9, 144.3)
Routing:
- net +BATT: track 258.2 -> 259.2 mm
- net Net-(C38-Pad2): track 109.2 -> 110.2 mm
- added copper zone on B.Cu, net +BATT
- removed copper zone on B.Cu, net VCC

Commit message: some changes
Parts:
- removed C16, C18, C5, C7: F_cap, Capacitors_SMD:C_0402
- removed C17, C6: Diff_Cap, Capacitors_SMD:C_0402
- removed C23: 1uF, Capacitors_SMD:C_0402
- removed C24: 10nF, Capacitors_SMD:C_0402
- removed C25: 100nF, Capacitors_SMD:C_0402
- removed C26: C_Small, Capacitors_SMD:C_0402
- removed M1: ANEOMETER, Wire_Connections_Bridges:WireConnection_2.00mmDrill
- removed MK5, MK6, MK7, MK8: Mounting_Hole_PAD, Measurement_Points:Measurement_Point_Square-SMD-Pad_Big
- removed R1, R10, R13, R6: 10MΩ, Resistors_SMD:R_0603
- removed R11, R12, R4, R5: 510Ω, Resistors_SMD:R_0603
- removed R21: 100kΩ, Resistors_SMD:R_0603
- removed U2: ADS1120-PW, Housings_SSOP:TSSOP-16_4.4x5mm_Pitch0.65mm
- removed U5: MPL115A1, Housings_LGA:LGA-8_3x5mm_Pitch1.25mm
- removed U6: MPU-9250, Housings_DFN_QFN:QFN-24-1EP_3x3mm_Pitch0.4mm
- J2: value Conn_02x10_Odd_Even -> Conn_01x06; footprint Pin_Headers:Pin_Header_Straight_2x10_Pitch2.54mm -> Pin_Headers:Pin_Header_Straight_1x06_Pitch2.54mm
- U1: value LT1129CS8-3.3 -> LT1129-3.3_SOT223; footprint Power_Integrations:SO-8C -> TO_SOT_Packages_SMD:SOT-223-3Lead_TabPin2
- moved J2 8.65 mm to (124.2, 59.4)
- moved C29 1.27 mm to (58.7, 89.9)
- moved Y2 1.08 mm to (58.7, 92.7)
- moved C30 0.92 mm to (58.7, 95.5)
Connections:
- AE1 pad 2: Net-(AE1-Pad2) -> (no net)
- DRA1 pad 11: Net-(DRA1-Pad11) -> (no net)
- DRA1 pad 13: Net-(DRA1-Pad13) -> (no net)
- DRA1 pad 14: Net-(DRA1-Pad14) -> (no net)
- DRA1 pad 15: Net-(DRA1-Pad15) -> (no net)
- DRA1 pad 2: Net-(DRA1-Pad2) -> (no net)
- DRA1 pad 4: Net-(DRA1-Pad4) -> (no net)
- J2 pad 2: GND -> (no net)
- J2 pad 3: SWCLK -> (no net)
- J2 pad 4: GND -> (no net)
- J2 pad 5: SWO -> (no net)
- U1 pad 1: +3V3 -> +BATT
- U1 pad 2: +3V3 -> GND
- U3 pad 10: ANEOMETER -> (no net)
- U3 pad 11: Net-(U3-Pad11) -> (no net)
- U3 pad 12: Net-(U3-Pad12) -> (no net)
- U3 pad 21: SWO -> (no net)
- U3 pad 22: Net-(U3-Pad22) -> (no net)
- U3 pad 23: Net-(U3-Pad23) -> (no net)
- U3 pad 24: RESET -> (no net)
- U3 pad 25: SWCLK -> (no net)
- U3 pad 26: SWDIO -> (no net)
- U3 pad 32: Net-(U3-Pad32) -> (no net)
- U3 pad 37: CS_ADS1120 -> (no net)
- U3 pad 38: SPI_CLK -> (no net)
- U3 pad 39: CS_MPL115A1 -> (no net)
- U3 pad 40: SHDMPL115A1 -> (no net)
- U3 pad 41: SPI_MSO -> (no net)
- U3 pad 42: SPI_MSI -> (no net)
- U3 pad 43: SPI_DRDY -> (no net)
- U3 pad 44: Net-(U3-Pad44) -> (no net)
- U3 pad 6: Net-(U3-Pad6) -> (no net)
- U3 pad 8: Net-(U3-Pad8) -> (no net)
- U3 pad 9: Net-(U3-Pad9) -> (no net)
Routing:
- net +3V3: track 328.0 -> 2.89 mm
- net (no net): track 6.00 -> 256.8 mm
- net GND: track 518.6 -> 423.6 mm, vias 66 -> 51
- net SWDIO: track 73.5 -> 0.00 mm
- net RESET: track 73.4 -> 0.00 mm
- net SWO: track 71.1 -> 0.00 mm
- net SWCLK: track 64.1 -> 0.00 mm
- net ANEOMETER: track 44.7 -> 0.00 mm
- net SPI_MSO: track 37.8 -> 0.00 mm
- net SPI_MSI: track 33.3 -> 0.00 mm
- net CS_ADS1120: track 32.8 -> 0.00 mm
- net SPI_CLK: track 31.3 -> 0.00 mm
- net SPI_DRDY: track 21.4 -> 0.00 mm
- net CS_MPL115A1: track 18.9 -> 0.00 mm
- net SHDMPL115A1: track 17.2 -> 0.00 mm
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